File: rs232usb/kicad/rs232usb.kicad_sch (KiCad schematic)
At the start: 13 parts, among them J1 USB_C_Receptacle_USB2.0_14P, J2 DE9_Socket, U1 CH340N, U2 MAX232

Commit message: Fix rs232usb wrong MAX232 setup
Parts:
- removed C2, C3, C4: 22u, Capacitor_Tantalum_SMD:CP_EIA-3528-12_Kemet-T, symbol Device:C_Polarized
- added C10, C7, C8, C9: 1u, Capacitor_SMD:C_0805_2012Metric, symbol Device:C
Connections:
- net GND: now also C10.1, C9.1
- net at U2.2 (VS+): now also C9.2
- net at U2.6 (VS-): now also C10.2
- net at U2.4 (C2+): now also C8.2
- net at U2.5 (C2-): now also C8.1
- net at U2.1 (C1+): now also C7.1
- net at U2.3 (C1-): now also C7.2
Other:
- moved on the sheet: C1, C5, C6, H1, J1, J2, R1, R2, U1, U2
