File: skadis_clock/kicad/digit.kicad_sch (KiCad schematic)
At the start: 21 parts

Commit message: skadis_clock: Add initial FW (based on ledclock)
Other:
- company: (none) -> A. K.
- title: (none) -> SKADIS LED clock digit
Changed lines of the file:
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@@
 	(generator_version "9.0")
 	(paper "A4")
+	(title_block
+		(title "SKADIS LED clock digit")
+		(date "2025-10-11")
+		(rev "A")
+		(company "A. K.")
+	)
 	(junction
 		(at 140.97 114.3)
