File: skadis_clock/kicad/skadis_clock.kicad_sch (KiCad schematic)
At the start: 28 parts, among them J1 AVR-ISP-6, J2 USB_C_Receptacle_PowerOnly_6P, Q1 BC807, Q2 BC807, Q3 BC807, Q4 BC807, SW1 SW_Push, SW2 SW_Push, U1 ATtiny2313-20S, Y1 Crystal

Commit message: skadis_clock: Add initial FW (based on ledclock)
Other:
- company: (none) -> A. K.
- title: (none) -> SKADIS LED clock
Changed lines of the file:
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@@
 	(generator_version "9.0")
 	(paper "A4")
+	(title_block
+		(title "SKADIS LED clock")
+		(date "2025-10-11")
+		(rev "A")
+		(company "A. K.")
+	)
 	(junction
 		(at 189.23 106.68)
